File: totem_0_3.kicad_sch (KiCad schematic)
At the start: 46 parts, among them J1 MJ-4PP-9, J2 MJ-4PP-9, J3 SS-52400-003, J4 SS-52400-003, U3 RP2040, U4 RP2040

Commit message: Improve spacing
Other:
- note added: "LEFT"
- note added: "RIGHT"
- note removed: "L E F T"
- note removed: "R I G H T"
- moved on the sheet: RSW1, RSW2
Changed lines of the file:
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@@
 	)
 	(rectangle
-		(start 86.36 78.74)
-		(end 116.84 96.52)
+		(start 96.52 81.28)
+		(end 127 99.06)
 		(stroke
 			(width 0)
@@
 	)
 	(rectangle
-		(start 187.96 76.2)
-		(end 218.44 93.98)
+		(start 172.72 81.28)
+		(end 203.2 99.06)
 		(stroke
 			(width 0)
@@
 	(text "R E S E T \nB U T T O N"
 		(exclude_from_sim no)
-		(at 87.122 95.25 0)
+		(at 97.282 97.79 0)
 		(effects
 			(font
@@
 	(text "R E S E T \nB U T T O N"
 		(exclude_from_sim no)
-		(at 188.976 92.456 0)
+		(at 173.736 97.536 0)
 		(effects
 			(font
@@
 		)
 	)
-	(text "R I G H T"
+	(text "RIGHT"
 		(exclude_from_sim no)
 		(at 149.098 89.916 0)
@@
 		)
 	)
-	(text "L E F T"
+	(text "LEFT"
 		(exclude_from_sim no)
 		(at 146.304 90.17 0)
@@
 	(global_label "GND_L"
 		(shape input)
-		(at 107.95 86.36 0)
+		(at 118.11 88.9 0)
 		(fields_autoplaced yes)
 		(effects
@@
 		)
 		(property "Intersheetrefs" "${INTERSHEET_REFS}"
-			(at 116.2293 86.2806 0)
+			(at 126.3893 88.8206 0)
 			(effects
 				(font
@@
 	(global_label "RESET_R"
 		(shape input)
-		(at 199.39 83.82 180)
+		(at 184.15 88.9 180)
 		(fields_autoplaced yes)
 		(effects
@@
 		)
 		(property "Intersheetrefs" "${INTERSHEET_REFS}"
-			(at 188.994 83.7406 0)
+			(at 173.754 88.8206 0)
 			(effects
 				(font
@@
 	(global_label "RESET_L"
 		(shape input)
-		(at 97.79 86.36 180)
+		(at 107.95 88.9 180)
 		(fields_autoplaced yes)
 		(effects
@@
 		)
 		(property "Intersheetrefs" "${INTERSHEET_REFS}"
-			(at 87.6359 86.4394 0)
+			(at 97.7959 88.9794 0)
 			(effects
 				(font
@@
 	(global_label "GND_R"
 		(shape input)
-		(at 209.55 83.82 0)
+		(at 194.31 88.9 0)
 		(fields_autoplaced yes)
 		(effects
@@
 		)
 		(property "Intersheetrefs" "${INTERSHEET_REFS}"
-			(at 218.0712 83.7406 0)
+			(at 202.8312 88.8206 0)
 			(effects
 				(font
@@
 	(symbol
 		(lib_id "Switch:SW_Push")
-		(at 102.87 86.36 0)
+		(at 113.03 88.9 0)
 		(unit 1)
 		(exclude_from_sim no)
@@
 		(fields_autoplaced yes)
 		(property "Reference" "RSW1"
-			(at 102.87 80.518 0)
+			(at 113.03 83.058 0)
 			(effects
 				(font
@@
 		)
 		(property "Value" "SW_Push"
-			(at 102.87 80.518 0)
+			(at 113.03 83.058 0)
 			(effects
 				(font
@@
 		)
 		(property "Footprint" "TOTEMlib:SKHLLCA010"
-			(at 102.87 81.28 0)
+			(at 113.03 83.82 0)
 			(effects
 				(font
@@
 		)
 		(property "Datasheet" "~"
-			(at 102.87 81.28 0)
+			(at 113.03 83.82 0)
 			(effects
 				(font
@@
 		)
 		(property "Description" ""
-			(at 102.87 86.36 0)
+			(at 113.03 88.9 0)
 			(effects
 				(font
@@
 	(symbol
 		(lib_id "Switch:SW_Push")
-		(at 204.47 83.82 0)
+		(at 189.23 88.9 0)
 		(unit 1)
 		(exclude_from_sim no)
@@
 		(fields_autoplaced yes)
 		(property "Reference" "RSW2"
-			(at 204.47 78.486 0)
+			(at 189.23 83.566 0)
 			(effects
 				(font
@@
 		)
 		(property "Value" "SW_Push"
-			(at 204.47 77.978 0)
+			(at 189.23 83.058 0)
 			(effects
 				(font
@@
 		)
 		(property "Footprint" "TOTEMlib:SKHLLCA010"
-			(at 204.47 78.74 0)
+			(at 189.23 83.82 0)
 			(effects
 				(font
@@
 		)
 		(property "Datasheet" "~"
-			(at 204.47 78.74 0)
+			(at 189.23 83.82 0)
 			(effects
 				(font
@@
 		)
 		(property "Description" ""
-			(at 204.47 83.82 0)
+			(at 189.23 88.9 0)
 			(effects
 				(font

Commit message: better spacing in schema
Parts:
- renumbered J3 to LJ1, RSW1 to LRSW1, J4 to RJ1, RSW2 to RRSW1
Other:
- moved on the sheet: RJ1
Changed lines of the file:
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@@
 	(symbol
 		(lib_id "USB-C-SS:SS-52400-003")
-		(at 176.53 124.46 0)
+		(at 179.07 124.46 0)
 		(unit 1)
 		(exclude_from_sim no)
@@
 		(dnp no)
 		(fields_autoplaced yes)
-		(property "Reference" "J4"
-			(at 176.53 101.6 0)
+		(property "Reference" "RJ1"
+			(at 179.07 101.6 0)
 			(effects
 				(font
@@
 		)
 		(property "Value" "SS-52400-003"
-			(at 176.53 104.14 0)
+			(at 179.07 104.14 0)
 			(effects
 				(font
@@
 		)
 		(property "Footprint" "SS-52400-003:BELFUSE_SS-52400-003"
-			(at 176.53 124.46 0)
+			(at 179.07 124.46 0)
 			(effects
 				(font
@@
 		)
 		(property "Datasheet" "${KIPRJMOD}/datasheets/usb-c/dr-stw-ss-52400-003.pdf"
-			(at 176.53 124.46 0)
-			(effects
-				(font
-					(size 1.27 1.27)
-				)
-				(hide yes)
-			)
-		)
-		(property "Description" ""
-			(at 176.53 124.46 0)
+			(at 179.07 124.46 0)
+			(effects
+				(font
+					(size 1.27 1.27)
+				)
+				(hide yes)
+			)
+		)
+		(property "Description" ""
+			(at 179.07 124.46 0)
 			(effects
 				(font
@@
 		)
 		(property "PARTREV" "A0"
-			(at 176.53 124.46 0)
+			(at 179.07 124.46 0)
 			(effects
 				(font
@@
 		)
 		(property "STANDARD" "Manufacturer Recommendations"
-			(at 176.53 124.46 0)
+			(at 179.07 124.46 0)
 			(effects
 				(font
@@
 		)
 		(property "MAXIMUM_PACKAGE_HEIGHT" "2.96 mm"
-			(at 176.53 124.46 0)
+			(at 179.07 124.46 0)
 			(effects
 				(font
@@
 		)
 		(property "MANUFACTURER" "BelFuse"
-			(at 176.53 124.46 0)
+			(at 179.07 124.46 0)
 			(effects
 				(font
@@
 		)
 		(property "Supplier" "https://www.digikey.co.za/en/products/detail/stewart-connector/SS-52400-003/11205655"
-			(at 176.53 124.46 0)
+			(at 179.07 124.46 0)
 			(effects
 				(font
@@
 			(project "totem_0_3"
 				(path "/4d1e609f-5432-4afb-8ee7-7d2d9aaaee48"
-					(reference "J4")
+					(reference "RJ1")
 					(unit 1)
 				)
@@
 		(dnp no)
 		(fields_autoplaced yes)
-		(property "Reference" "RSW1"
+		(property "Reference" "LRSW1"
 			(at 113.03 83.058 0)
 			(effects
@@
 			(project ""
 				(path "/4d1e609f-5432-4afb-8ee7-7d2d9aaaee48"
-					(reference "RSW1")
+					(reference "LRSW1")
 					(unit 1)
 				)
@@
 		(dnp no)
 		(fields_autoplaced yes)
-		(property "Reference" "RSW2"
-			(at 189.23 83.566 0)
+		(property "Reference" "RRSW1"
+			(at 189.23 83.82 0)
 			(effects
 				(font
@@
 			(project ""
 				(path "/4d1e609f-5432-4afb-8ee7-7d2d9aaaee48"
-					(reference "RSW2")
+					(reference "RRSW1")
 					(unit 1)
 				)
@@
 		(lib_id "USB-C-SS:SS-52400-003")
 		(at 118.11 124.46 0)
-		(unit 1)
-		(exclude_from_sim no)
-		(in_bom yes)
-		(on_board yes)
-		(dnp no)
-		(fields_autoplaced yes)
-		(property "Reference" "J3"
+		(mirror y)
+		(unit 1)
+		(exclude_from_sim no)
+		(in_bom yes)
+		(on_board yes)
+		(dnp no)
+		(property "Reference" "LJ1"
 			(at 118.11 101.6 0)
 			(effects
@@
 			(project ""
 				(path "/4d1e609f-5432-4afb-8ee7-7d2d9aaaee48"
-					(reference "J3")
-					(unit 1)
-				)
+					(reference "LJ1")
+					(unit 1)
+				)
